File: pcb/Boreas.kicad_pcb (KiCad board)
At the start: 2 copper layers, 93 parts, among them J1 USB_C_Receptacle_USB2.0_16P, J2 Screw_Terminal_01x02, J3 Conn_01x03, J4 Conn_01x03, J5 Conn_01x03, SW1 TS-1088-AR02016, SW2 TS-1088-AR02016, SW3 TS-1088-AR02016, SW4 TS-1088-AR02016, U1 BMP580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

Commit message: done!
Parts:
- J3, J4, J5: footprint Connector_PinHeader_2.54mm:PinHeader_2x03_P2.54mm_Vertical -> Connector_PinHeader_2.54mm:PinHeader_1x03_P2.54mm_Vertical
- moved R14 164.1 mm to (194.9, 72.3), turned to -90 degrees
- moved R25 163.7 mm to (197.3, 83.0), turned to 90 degrees
- moved R13 163.3 mm to (193.8, 72.3), turned to 90 degrees
- moved R24 162.2 mm to (195.2, 83.0), turned to 90 degrees
- moved J3 161.4 mm to (184.4, 103.5), turned to 180 degrees
- moved Card1 161.1 mm to (189.4, 65.3), turned to 180 degrees
- moved R23 160.9 mm to (193.4, 83.0), turned to 90 degrees
- moved C15 159.8 mm to (185.7, 91.4)
- moved R16 159.5 mm to (185.8, 93.5)
- moved R17 158.4 mm to (185.7, 92.4), turned to 180 degrees
- moved R22 158.1 mm to (191.9, 75.3), turned to 180 degrees
- moved R21 158.0 mm to (191.6, 72.3), turned to -90 degrees
- moved C16 156.8 mm to (183.5, 89.3), turned to 180 degrees
- moved R20 156.2 mm to (189.5, 72.3), turned to -90 degrees
- moved C38 155.9 mm to (191.7, 82.0)
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Routing:
- net +3V3: track 0.00 -> 192.8 mm, vias 0 -> 12
- net /SCL: track 0.00 -> 67.1 mm, vias 0 -> 4
- net /BUZZER: track 0.00 -> 62.3 mm, vias 0 -> 2
- net /SDA: track 0.00 -> 61.1 mm, vias 0 -> 4
- net VBUS: track 0.00 -> 58.7 mm, vias 0 -> 4
- net /LED_1: track 0.00 -> 54.8 mm, vias 0 -> 4
- net /LED_2: track 0.00 -> 52.9 mm, vias 0 -> 4
- net /SD_CD: track 0.00 -> 52.6 mm, vias 0 -> 4
- net /LED_3: track 0.00 -> 51.5 mm, vias 0 -> 4
- net /BQ_CE: track 0.00 -> 51.0 mm, vias 0 -> 2
- net VSYS: track 0.00 -> 50.3 mm, vias 0 -> 3
- net /SD_CMD: track 0.00 -> 50.1 mm, vias 0 -> 4
- net /BTN_1: track 0.00 -> 49.0 mm, vias 0 -> 4
- net /BMP_INT: track 0.00 -> 48.8 mm, vias 0 -> 2
- net /SD_CLK: track 0.00 -> 46.5 mm, vias 0 -> 2
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- added copper zone on B.Cu, net GND
- added copper zone on F.Cu, net GND
Other:
- board outline added: 50 x 50 mm
