File: pcb/Boreas.kicad_sch (KiCad schematic)
At the start: 93 parts, among them J1 USB_C_Receptacle_USB2.0_16P, J2 Screw_Terminal_01x02, J3 Conn_01x03, J4 Conn_01x03, J5 Conn_01x03, SW1 TS-1088-AR02016, SW2 TS-1088-AR02016, SW3 TS-1088-AR02016, SW4 TS-1088-AR02016, U1 BMP580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

Commit message: done!
Parts:
- J3, J4, J5: footprint Connector_PinHeader_2.54mm:PinHeader_2x03_P2.54mm_Vertical -> Connector_PinHeader_2.54mm:PinHeader_1x03_P2.54mm_Vertical
Changed lines of the file:
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@@
 	)
 	(symbol
-		(lib_id "Connector_Generic:Conn_01x03")
-		(at 317.5 204.47 0)
-		(unit 1)
-		(exclude_from_sim no)
-		(in_bom yes)
-		(on_board yes)
-		(dnp no)
-		(fields_autoplaced yes)
-		(property "Reference" "J4"
-			(at 320.04 203.1999 0)
-			(effects
-				(font
-					(size 1.27 1.27)
-				)
-				(justify left)
-			)
-		)
-		(property "Value" "Conn_01x03"
-			(at 320.04 205.7399 0)
-			(effects
-				(font
-					(size 1.27 1.27)
-				)
-				(justify left)
-			)
-		)
-		(property "Footprint" "Connector_PinHeader_2.54mm:PinHeader_2x03_P2.54mm_Vertical"
-			(at 317.5 204.47 0)
-			(effects
-				(font
-					(size 1.27 1.27)
-				)
-				(hide yes)
-			)
-		)
-		(property "Datasheet" "~"
-			(at 317.5 204.47 0)
-			(effects
-				(font
-					(size 1.27 1.27)
-				)
-				(hide yes)
-			)
-		)
-		(property "Description" "Generic connector, single row, 01x03, script generated (kicad-library-utils/schlib/autogen/connector/)"
-			(at 317.5 204.47 0)
-			(effects
-				(font
-					(size 1.27 1.27)
-				)
-				(hide yes)
-			)
-		)
-		(pin "3"
-		)
-		(pin "1"
-		)
-		(pin "2"
-		)
-		(instances
-			(project "Boreas"
-				(path "/66b324e0-ef0b-4e1e-b632-08b83dd1529e"
-					(reference "J4")
-					(unit 1)
-				)
-			)
-		)
-	)
-	(symbol
 		(lib_id "Device:LED")
 		(at 393.7 219.71 180)
@@
 	)
 	(symbol
+		(lib_id "Connector_Generic:Conn_01x03")
+		(at 317.5 222.25 0)
+		(unit 1)
+		(exclude_from_sim no)
+		(in_bom yes)
+		(on_board yes)
+		(dnp no)
+		(fields_autoplaced yes)
+		(property "Reference" "J5"
+			(at 320.04 220.9799 0)
+			(effects
+				(font
+					(size 1.27 1.27)
+				)
+				(justify left)
+			)
+		)
+		(property "Value" "Conn_01x03"
+			(at 320.04 223.5199 0)
+			(effects
+				(font
+					(size 1.27 1.27)
+				)
+				(justify left)
+			)
+		)
+		(property "Footprint" "Connector_PinHeader_2.54mm:PinHeader_1x03_P2.54mm_Vertical"
+			(at 317.5 222.25 0)
+			(effects
+				(font
+					(size 1.27 1.27)
+				)
+				(hide yes)
+			)
+		)
+		(property "Datasheet" "~"
+			(at 317.5 222.25 0)
+			(effects
+				(font
+					(size 1.27 1.27)
+				)
+				(hide yes)
+			)
+		)
+		(property "Description" "Generic connector, single row, 01x03, script generated (kicad-library-utils/schlib/autogen/connector/)"
+			(at 317.5 222.25 0)
+			(effects
+				(font
+					(size 1.27 1.27)
+				)
+				(hide yes)
+			)
+		)
+		(pin "3"
+		)
+		(pin "1"
+		)
+		(pin "2"
+		)
+		(instances
+			(project "Boreas"
+				(path "/66b324e0-ef0b-4e1e-b632-08b83dd1529e"
+					(reference "J5")
+					(unit 1)
+				)
+			)
+		)
+	)
+	(symbol
 		(lib_id "easyeda2kicad:TS-1088-AR02016")
 		(at 132.08 168.91 0)
@@
 	)
 	(symbol
-		(lib_id "Connector_Generic:Conn_01x03")
-		(at 317.5 222.25 0)
+		(lib_id "power:GND")
+		(at 311.15 207.01 0)
 		(unit 1)
 		(exclude_from_sim no)
@@
 		(dnp no)
 		(fields_autoplaced yes)
-		(property "Reference" "J5"
-			(at 320.04 220.9799 0)
+		(property "Reference" "#PWR053"
+			(at 311.15 213.36 0)
 			(effects
 				(font
-					(size 1.27 1.27)
+					(size 0.762 0.762)
 				)
-				(justify left)
+				(hide yes)
 			)
 		)
-		(property "Value" "Conn_01x03"
-			(at 320.04 223.5199 0)
+		(property "Value" "GND"
+			(at 311.15 212.09 0)
 			(effects
 				(font
-					(size 1.27 1.27)
+					(size 0.762 0.762)
 				)
-				(justify left)
 			)
 		)
-		(property "Footprint" "Connector_PinHeader_2.54mm:PinHeader_2x03_P2.54mm_Vertical"
-			(at 317.5 222.25 0)
+		(property "Footprint" ""
+			(at 311.15 207.01 0)
 			(effects
 				(font
-					(size 1.27 1.27)
+					(size 0.762 0.762)
 				)
 				(hide yes)
 			)
 		)
-		(property "Datasheet" "~"
-			(at 317.5 222.25 0)
+		(property "Datasheet" ""
+			(at 311.15 207.01 0)
 			(effects
 				(font
-					(size 1.27 1.27)
+					(size 0.762 0.762)
 				)
 				(hide yes)
 			)
 		)
-		(property "Description" "Generic connector, single row, 01x03, script generated (kicad-library-utils/schlib/autogen/connector/)"
-			(at 317.5 222.25 0)
+		(property "Description" "Power symbol creates a global label with name \"GND\" , ground"
+			(at 311.15 207.01 0)
 			(effects
 				(font
-					(size 1.27 1.27)
+					(size 0.762 0.762)
 				)
 				(hide yes)
 			)
 		)
-		(pin "3"
-		)
 		(pin "1"
 		)
-		(pin "2"
-		)
 		(instances
 			(project "Boreas"
 				(path "/66b324e0-ef0b-4e1e-b632-08b83dd1529e"
-					(reference "J5")
+					(reference "#PWR053")
 					(unit 1)
 				)
@@
 	)
 	(symbol
-		(lib_id "power:GND")
-		(at 311.15 207.01 0)
+		(lib_id "Device:C")
+		(at 20.32 262.89 180)
 		(unit 1)
 		(exclude_from_sim no)
@@
 		(on_board yes)
 		(dnp no)
-		(fields_autoplaced yes)
-		(property "Reference" "#PWR053"
-			(at 311.15 213.36 0)
+		(property "Reference" "C21"
+			(at 25.654 263.906 0)
 			(effects
 				(font
 					(size 0.762 0.762)
 				)
-				(hide yes)
+				(justify left)
 			)
 		)
-		(property "Value" "GND"
-			(at 311.15 212.09 0)
+		(property "Value" "0.1uF"
+			(at 26.162 262.128 0)
 			(effects
 				(font
 					(size 0.762 0.762)
 				)
+				(justify left)
 			)
 		)
-		(property "Footprint" ""
-			(at 311.15 207.01 0)
+		(property "Footprint" "Capacitor_SMD:C_0402_1005Metric"
+			(at 19.3548 259.08 0)
 			(effects
 				(font
@@
 			)
 		)
-		(property "Datasheet" ""
-			(at 311.15 207.01 0)
+		(property "Datasheet" "~"
+			(at 20.32 262.89 0)
 			(effects
 				(font
@@
 			)
 		)
-		(property "Description" "Power symbol creates a global label with name \"GND\" , ground"
-			(at 311.15 207.01 0)
+		(property "Description" "Unpolarized capacitor"
+			(at 20.32 262.89 0)
 			(effects
 				(font
@@
 			)
 		)
+		(pin "2"
+		)
 		(pin "1"
 		)
@@
 			(project "Boreas"
 				(path "/66b324e0-ef0b-4e1e-b632-08b83dd1529e"
-					(reference "#PWR053")
+					(reference "C21")
 					(unit 1)
 				)
@@
 	)
 	(symbol
-		(lib_id "Device:C")
-		(at 20.32 262.89 180)
+		(lib_id "Connector_Generic:Conn_01x03")
+		(at 317.5 187.96 0)
 		(unit 1)
 		(exclude_from_sim no)
@@
 		(on_board yes)
 		(dnp no)
-		(property "Reference" "C21"
-			(at 25.654 263.906 0)
+		(fields_autoplaced yes)
+		(property "Reference" "J3"
+			(at 320.04 186.6899 0)
 			(effects
 				(font
-					(size 0.762 0.762)
+					(size 1.27 1.27)
 				)
 				(justify left)
 			)
 		)
-		(property "Value" "0.1uF"
-			(at 26.162 262.128 0)
+		(property "Value" "Conn_01x03"
+			(at 320.04 189.2299 0)
 			(effects
 				(font
-					(size 0.762 0.762)
+					(size 1.27 1.27)
 				)
 				(justify left)
 			)
 		)
-		(property "Footprint" "Capacitor_SMD:C_0402_1005Metric"
-			(at 19.3548 259.08 0)
+		(property "Footprint" "Connector_PinHeader_2.54mm:PinHeader_1x03_P2.54mm_Vertical"
+			(at 317.5 187.96 0)
 			(effects
 				(font
-					(size 0.762 0.762)
+					(size 1.27 1.27)
 				)
 				(hide yes)
@@
 		)
 		(property "Datasheet" "~"
-			(at 20.32 262.89 0)
+			(at 317.5 187.96 0)
 			(effects
 				(font
-					(size 0.762 0.762)
+					(size 1.27 1.27)
 				)
 				(hide yes)
 			)
 		)
-		(property "Description" "Unpolarized capacitor"
-			(at 20.32 262.89 0)
+		(property "Description" "Generic connector, single row, 01x03, script generated (kicad-library-utils/schlib/autogen/connector/)"
+			(at 317.5 187.96 0)
 			(effects
 				(font
-					(size 0.762 0.762)
+					(size 1.27 1.27)
 				)
 				(hide yes)
 			)
 		)
-		(pin "2"
+		(pin "3"
 		)
 		(pin "1"
 		)
+		(pin "2"
+		)
 		(instances
-			(project "Boreas"
+			(project ""
 				(path "/66b324e0-ef0b-4e1e-b632-08b83dd1529e"
-					(reference "C21")
+					(reference "J3")
 					(unit 1)
 				)
@@
 	(symbol
 		(lib_id "Connector_Generic:Conn_01x03")
-		(at 317.5 187.96 0)
+		(at 317.5 204.47 0)
 		(unit 1)
 		(exclude_from_sim no)
@@
 		(dnp no)
 		(fields_autoplaced yes)
-		(property "Reference" "J3"
-			(at 320.04 186.6899 0)
+		(property "Reference" "J4"
+			(at 320.04 203.1999 0)
 			(effects
 				(font
@@
 		)
 		(property "Value" "Conn_01x03"
-			(at 320.04 189.2299 0)
+			(at 320.04 205.7399 0)
 			(effects
 				(font
@@
 			)
 		)
-		(property "Footprint" "Connector_PinHeader_2.54mm:PinHeader_2x03_P2.54mm_Vertical"
-			(at 317.5 187.96 0)
+		(property "Footprint" "Connector_PinHeader_2.54mm:PinHeader_1x03_P2.54mm_Vertical"
+			(at 317.5 204.47 0)
 			(effects
 				(font
@@
 		)
 		(property "Datasheet" "~"
-			(at 317.5 187.96 0)
+			(at 317.5 204.47 0)
 			(effects
 				(font
@@
 		)
 		(property "Description" "Generic connector, single row, 01x03, script generated (kicad-library-utils/schlib/autogen/connector/)"
-			(at 317.5 187.96 0)
+			(at 317.5 204.47 0)
 			(effects
 				(font
@@
 		)
 		(instances
-			(project ""
+			(project "Boreas"
 				(path "/66b324e0-ef0b-4e1e-b632-08b83dd1529e"
-					(reference "J3")
+					(reference "J4")
 					(unit 1)
 				)
